File: ExpansionBoards/ATX-PSU_8b/ATX-PSU_8b.kicad_pcb (KiCad board)
At the start: 2 copper layers, 99.1 x 99.1 mm, 49 parts, among them J1 39-30-1240, J2 Phoenix 3,5mm, J3 Conn_02x05_Odd_Even, J4 Conn_02x20_Odd_Even, J5 Conn_02x20_Odd_Even, J6 Conn_01x06, Q1 PN2222A, Q2 PN2222A, SW2 SW_Push, U1 74LS74

Commit message: Cherry-pick from cleanup archive
Parts:
- removed C3: 100nF, Capacitor_THT:C_Disc_D4.3mm_W1.9mm_P5.00mm
Routing:
- net /PWR-SW-R: track 29.4 -> 14.1 mm
Other:
- board text removed: "C3"
